File: lab8/pcb.kicad_sch (KiCad schematic)
At the start: 11 parts

Commit message: Added lab8
Parts:
- removed R1, R2, RH, RL, RSafe: (no value), symbol Device:R
- removed U?: (no value), symbol Amplifier_Operational:TLC277
- added R1: 6.7k, Resistor_THT:R_Axial_DIN0207_L6.3mm_D2.5mm_P15.24mm_Horizontal, symbol Device:R_US
- added R2: 2k, Resistor_THT:R_Axial_DIN0207_L6.3mm_D2.5mm_P15.24mm_Horizontal, symbol Device:R_US
- added R3: 390k, Resistor_THT:R_Axial_DIN0207_L6.3mm_D2.5mm_P15.24mm_Horizontal, symbol Device:R_US
- added R4: 1k, Resistor_THT:R_Axial_DIN0207_L6.3mm_D2.5mm_P15.24mm_Horizontal, symbol Device:R_US
- added R5: 100, Resistor_THT:R_Axial_DIN0207_L6.3mm_D2.5mm_P15.24mm_Horizontal, symbol Device:R_US
- added Rf1, Rl1: (no value), symbol Device:R_US
- added U1: TLC277, Package_DIP:DIP-8_W7.62mm, symbol Amplifier_Operational:TLC277
- added U2: (no value), symbol dk_Optical-Sensors-Reflective-Analog-Output:QRD1114
- CH1: renamed from CH; value (none) -> 47u; footprint (none) -> Capacitor_THT:CP_Axial_L10.0mm_D4.5mm_P15.00mm_Horizontal
- CL1: renamed from CL; value (none) -> 47u; footprint (none) -> Capacitor_THT:CP_Axial_L10.0mm_D4.5mm_P15.00mm_Horizontal
- D1, D2: renamed from D?; value (none) -> 1N5817; footprint (none) -> Diode_THT:D_DO-41_SOD81_P10.16mm_Horizontal
- J1: value (none) -> Conn_01x04_Male
Connections:
- net at J1.1 (Pin_1): now also Rf1.1, Rl1.1; no longer CH1.1
- net at D1.2 (A), D2.1 (K), J1.4 (Pin_4): now also R5.2
- net at CH1.2: now also R1.1, R2.1
- net at CL1.1: now also R2.2, U1.3 (+)
- net GND: no longer names the net of CL1.2, D2.2 (A), J1.2 (Pin_2)
- net GND: now also R1.2, R4.2, U2.2, U2.4
- new net: R3.1, R5.1, U1.1
- new net: CH1.1, Rl1.2, U2.1
- new net: R3.2, R4.1, U1.2 (-)
- new net: Rf1.2, U2.3

Commit message: Finished lab8
Parts:
- J1: footprint (none) -> Connector_PinHeader_2.54mm:PinHeader_1x04_P2.54mm_Vertical
- Rf1: value (none) -> 65; footprint (none) -> Resistor_THT:R_Axial_DIN0207_L6.3mm_D2.5mm_P15.24mm_Horizontal
- Rl1: value (none) -> 20k; footprint (none) -> Resistor_THT:R_Axial_DIN0207_L6.3mm_D2.5mm_P15.24mm_Horizontal
- U1: value TLC277 -> (none); footprint Package_DIP:DIP-8_W7.62mm -> (none)
- U2: value (none) -> QRD1114; footprint (none) -> digikey-footprints:Reflective_Sensor_QRD1114
Other:
- moved on the sheet: CH1, CL1, D1, R1, R2, R3, Rf1, Rl1
